File: Schematic/ecu.kicad_sch (KiCad schematic)
At the start: 10 parts, among them K1 Relay_SPST-NO, Q1 NMOS, SW1 SW_SPST, SW2 SW_SPST, U1 RP2040, U2 A1363xKTTN-1, U3 74LVC2T45DC

Commit message: this project is done (probably)
Parts:
- removed BT1: Battery_Cell, symbol Device:Battery_Cell
- removed K1: Relay_SPST-NO, symbol Relay:Relay_SPST-NO
- removed Q1: NMOS, symbol Simulation_SPICE:NMOS
- removed U1: RP2040, Package_DFN_QFN:QFN-56-1EP_7x7mm_P0.4mm_EP3.2x3.2mm, symbol MCU_RaspberryPi:RP2040
- removed U3: 74LVC2T45DC, Package_SO:VSSOP-8_2.3x2mm_P0.5mm, symbol Logic_LevelTranslator:74LVC2T45DC
- added A1: RaspberryPi_Pico, Module:RaspberryPi_Pico_Common_Unspecified, symbol MCU_Module:RaspberryPi_Pico
- added BT1: 12V Car Battery, symbol Device:Battery
- added C1, C3: 1uF, symbol Device:C
- added D1, D2: D, symbol Device:D
- added J1: OLED_128x64, symbol Connector:Conn_01x04_Socket
- added J2: Ignition Cutoff, symbol Connector:Conn_01x02_Socket
- added J3: MPX5700ASX, symbol Connector:Conn_01x06_Socket
- added K1, K2: Fujitsu_FTR-LYAA005x, Relay_THT:Relay_SPST-NO_Fujitsu_FTR-LYAA005x_FormA_Vertical, symbol Relay:Fujitsu_FTR-LYAA005x
- added M1: Fuel_Pump, symbol Motor:Motor_DC
- added M2: Motor_DC, symbol Motor:Motor_DC
- added Q1: NPN, symbol Simulation_SPICE:NPN
- added Q2: IRLZ44N, Package_TO_SOT_THT:TO-220-3_Vertical, symbol Transistor_FET:IRLZ44N
- added R12, R6: 10k, symbol Device:R
- added R3: 1k, symbol Device:R
- added R4: 1.8k, symbol Device:R
- added R5, R8: 3.3k, symbol Device:R
- added R7, R9: 5.6k, symbol Device:R
- added RV1: 10k Linear, symbol Device:R_Potentiometer
- added SW3: SW_SPST, symbol Switch:SW_SPST
- added TH1: Thermistor, symbol Device:Thermistor
- added U1: LM311, symbol Comparator:LM311
- added U3: Buck Converter, Module:Texas_EUS_R-PDSS-T5_THT, symbol Converter_DCDC:PTN78000H_EUS-5
- R1: value 10K -> 3.3k
- R2: value 220 -> 10k
- U2: value A1363xKTTN-1 -> OH49E
Connections:
- net OUT is gone; now on net +5V: SW2.1 (A)
- net +12V: now also R2.2, BT1.1 (+), K1.A2, K2.A2, U3.2 (VI)
- net +5V: now also SW1.1 (A), A1.40 (VBUS), C1.1, C3.1, J3.3 (Pin_3), R4.1, R6.2, U1.8 (V+), U3.5 (VO); no longer SW1.2 (B)
- net GND: now also A1.13 (GND), A1.18 (GND), A1.23 (GND), A1.28 (GND), A1.3 (GND), A1.33 (AGND), A1.38 (GND), A1.8 (GND), BT1.2 (-), C1.2, C3.2, D1.1 (K), J1.1 (GND), J3.2 (Pin_2), K1.14, K2.14, M1.2 (-), Q1.3 (E), Q2.3 (S), R12.1, R5.2, R7.1, R9.2, RV1.3, U1.1 (GND), U1.4 (V-), U3.1 (GND); no longer SW2.2 (B)
- net at U2.2 (VOUT): now also U1.2 (+)
- net at R2.1: now also Q1.1 (C), Q2.1 (G); no longer R1.1
- net at R1.2: now also J3.1 (Pin_1)
- new net: R4.2, R5.1, U1.3 (-)
- new net: J2.1 (Pin_1), SW3.1 (A)
- new net: J2.2 (Pin_2), SW3.2 (B)
- new net: R6.1, R8.2, U1.7
- new net: D1.2 (A), K1.A1, M1.1 (+)
- new net: D2.1 (K), M2.2 (-), Q2.2 (D)
- new net: D2.2 (A), K2.A1, M2.1 (+)
- new net: Q1.2 (B), R3.2
- new net: K2.13, SW2.2 (B)
- new net: K1.13, SW1.2 (B)
- new net +3.3V: A1.36 (3V3), J1.2 (VCC), RV1.1, TH1.2
- new net AFR_KNOB: A1.31 (GPIO26_ADC0), RV1.2
- new net HALL: A1.26 (GPIO20), R7.2, R8.1
- new net INJECTOR: A1.27 (GPIO21), R3.1
- new net MAP: A1.32 (GPIO27_ADC1), R1.1, R9.1
- new net SCL: A1.2 (GPIO1), J1.4 (SDA)
- new net SDA: A1.1 (GPIO0), J1.3 (SCL)
- new net TEMP: A1.34 (GPIO28_ADC2), R12.2, TH1.1
- no-connect marks 2 -> 28
Other:
- note added: "Air Fuel Ratio Control"
- note added: "Battery and 5V Converter"
- note added: "Fuel Pump"
- note added: "Hall Effect Sensor"
- note added: "Injector Firing System"
- note added: "Intake Air Temp"
- note added: "OLED Display"
- note added: "Pi Pico"
- note removed: "12V-5V Buck"
- note removed: "Injector"
- note removed: "Pump"
- company: (none) -> Brian Hill (@TrojanPinata)
- title: (none) -> PicoECU - Pi Pico Based ECU for Small Engines
